File: pcb/argo-v9-stable/argo-v9-stable-rev2/argo-v9-stable-rev2.kicad_sch (KiCad schematic)
At the start: 91 parts, among them IC1 MP2672GD, J1 Sparkfun_NEO-N9M-SMA, J2 USB4125-GF-A, J3 LED_power_button_RGB_LED, K1 PRL3-5V-DC-1A, Q2 BSD840N, SW1 POW, U1 orange_pi_zero_2w_2GB, U2 MAX11612, U3 CH221K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

Commit message: add datasheet and sparkfun links for GPS
Parts:
- J1: Hookup guide (none) -> https://learn.sparkfun.com/tutorials/sparkfun-gps-neo-m9n-h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; Ordering (none) -> https://www.sparkfun.com/sparkfun-gps-breakout-neo-m9n-sma-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
Changed lines of the file:
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@@
 			)
 		)
-		(property "Datasheet" "~"
+		(property "Datasheet" "https://cdn.sparkfun.com/assets/learn_tutorials/1/1/0/2/NEO-M9N-00B_DataSheet_UBX-19014285.pdf"
 			(at 127 19.05 0)
 			(effects
@@
 			(at 127 19.05 0)
 			(effects
+				(font
+					(size 1.27 1.27)
+				)
+				(hide yes)
+			)
+		)
+		(property "Ordering" "https://www.sparkfun.com/sparkfun-gps-breakout-neo-m9n-sma-qwiic.html"
+			(at 127 19.05 0)
+			(effects
+				(font
+					(size 1.27 1.27)
+				)
+				(hide yes)
+			)
+		)
+		(property "Hookup guide" "https://learn.sparkfun.com/tutorials/sparkfun-gps-neo-m9n-hookup-guide"
+			(at 127 19.05 0)
+			(effects
